Commit message: Edit meshes and description

File: goliath_description/urdf/goliath_model.urdf (robot description, URDF)
Before this commit: robot goliath, 9 links, 8 joints
Links:
- removed link rf_coxa_link
- removed link rf_femur_link
- removed link rf_tarsus_link
- removed link rf_tibia_link
- removed link upper_shassi_link
- added link body_link; visual mesh filename=package://goliath_description/meshes/body.stl scale=0.001 0.001 0.001
- link lf_coxa_link: geometry visual mesh filename=package://goliath_description/meshes/coxa.stl scale=0.001 0.001 0.001
- link lf_femur_link: geometry visual mesh filename=package://goliath_description/meshes/femur.stl scale=0.001 0.001 0.001
- link lf_tarsus_link: geometry visual mesh filename=package://goliath_description/meshes/leg_end.stl scale=0.001 0.001 0.001
- link lf_tibia_link: geometry visual mesh filename=package://goliath_description/meshes/tibia.stl scale=0.001 0.001 0.001
Joints:
- removed joint rf_coxa_joint
- removed joint rf_femur_joint
- removed joint rf_tarsus_joint
- removed joint rf_tibia_joint
- joint lf_coxa_joint: origin xyz=-0.063 0.092 0.00 rpy=0 0 2.18 -> xyz=-0.063 0.092 0.00 rpy=0 0 2.17; parent upper_shassi_link -> body_link

Commit message: Change goliath_locomotion.cpp for work with goliath_msgs Chage goliath_model.urdf - add second leg Fix bug with x and y coord in hexapod.cpp

File: goliath_description/urdf/goliath_model.urdf (robot description, URDF)
Before this commit: robot goliath, 5 links, 4 joints
Links:
- added link rf_coxa_link; visual mesh filename=package://goliath_description/meshes/coxa.stl scale=0.001 0.001 0.001
- added link rf_femur_link; visual mesh filename=package://goliath_description/meshes/femur.stl scale=0.001 0.001 0.001
- added link rf_tarsus_link; visual mesh filename=package://goliath_description/meshes/leg_end.stl scale=0.001 0.001 0.001
- added link rf_tibia_link; visual mesh filename=package://goliath_description/meshes/tibia.stl scale=0.001 0.001 0.001
Joints:
- added joint rf_coxa_joint: type revolute, parent body_link, child rf_coxa_link, origin xyz=0.063 0.092 0.00 rpy=0 0 0.6, axis 0 0 1, limit lower=-3.14 upper=3.14 effort=1.0 velocity=1.0
- added joint rf_femur_joint: type revolute, parent rf_coxa_link, child rf_femur_link, origin xyz=0.022 0.00 0.00 rpy=0 -0.785 0.0, axis 0 1 0, limit lower=-3.14 upper=3.14 effort=1.0 velocity=1.0
- added joint rf_tarsus_joint: type fixed, parent rf_tibia_link, child rf_tarsus_link, origin xyz=-0.115 0.0 0
- added joint rf_tibia_joint: type revolute, parent rf_femur_link, child rf_tibia_link, origin xyz=0.08 0.0 0.0 rpy=0 -0.785 0, axis 0 1 0, limit lower=-3.14 upper=3.14 effort=1.0 velocity=1.0

Commit message: Add 6 leg in goliath_model.urdf Corrected all CMakeLists.txt and package.xml

File: goliath_description/urdf/goliath_model.urdf (robot description, URDF)
Before this commit: robot goliath, 9 links, 8 joints
Links:
- added link lm_coxa_link; visual mesh filename=package://goliath_description/meshes/l_coxa.stl scale=0.001 0.001 0.001
- added link lm_femur_link; visual mesh filename=package://goliath_description/meshes/l_femur.stl scale=0.001 0.001 0.001
- added link lm_tarsus_link; visual mesh filename=package://goliath_description/meshes/leg_end.stl scale=0.001 0.001 0.001
- added link lm_tibia_link; visual mesh filename=package://goliath_description/meshes/l_tibia.stl scale=0.001 0.001 0.001
- added link lr_coxa_link; visual mesh filename=package://goliath_description/meshes/l_coxa.stl scale=0.001 0.001 0.001
- added link lr_femur_link; visual mesh filename=package://goliath_description/meshes/l_femur.stl scale=0.001 0.001 0.001
- added link lr_tarsus_link; visual mesh filename=package://goliath_description/meshes/leg_end.stl scale=0.001 0.001 0.001
- added link lr_tibia_link; visual mesh filename=package://goliath_description/meshes/l_tibia.stl scale=0.001 0.001 0.001
- added link rm_coxa_link; visual mesh filename=package://goliath_description/meshes/r_coxa.stl scale=0.001 0.001 0.001
- added link rm_femur_link; visual mesh filename=package://goliath_description/meshes/r_femur.stl scale=0.001 0.001 0.001
- added link rm_tarsus_link; visual mesh filename=package://goliath_description/meshes/leg_end.stl scale=0.001 0.001 0.001
- added link rm_tibia_link; visual mesh filename=package://goliath_description/meshes/r_tibia.stl scale=0.001 0.001 0.001
- added link rr_coxa_link; visual mesh filename=package://goliath_description/meshes/r_coxa.stl scale=0.001 0.001 0.001
- added link rr_femur_link; visual mesh filename=package://goliath_description/meshes/r_femur.stl scale=0.001 0.001 0.001
- added link rr_tarsus_link; visual mesh filename=package://goliath_description/meshes/leg_end.stl scale=0.001 0.001 0.001
- added link rr_tibia_link; visual mesh filename=package://goliath_description/meshes/r_tibia.stl scale=0.001 0.001 0.001
- link lf_coxa_link: geometry visual mesh filename=package://goliath_description/meshes/l_coxa.stl scale=0.001 0.001 0.001
- link lf_femur_link: geometry visual mesh filename=package://goliath_description/meshes/l_femur.stl scale=0.001 0.001 0.001
- link lf_tibia_link: geometry visual mesh filename=package://goliath_description/meshes/l_tibia.stl scale=0.001 0.001 0.001
- link rf_coxa_link: geometry visual mesh filename=package://goliath_description/meshes/r_coxa.stl scale=0.001 0.001 0.001
- link rf_femur_link: geometry visual mesh filename=package://goliath_description/meshes/r_femur.stl scale=0.001 0.001 0.001
- link rf_tibia_link: geometry visual mesh filename=package://goliath_description/meshes/r_tibia.stl scale=0.001 0.001 0.001
Joints:
- added joint lm_coxa_joint: type revolute, parent body_link, child lm_coxa_link, origin xyz=-0.072 0.0 0.0 rpy=0 0 3.14, axis 0 0 1, limit lower=-3.14 upper=3.14 effort=1.0 velocity=1.0
- added joint lm_femur_joint: type revolute, parent lm_coxa_link, child lm_femur_link, origin xyz=0.022 0.00 0.00 rpy=0 -0.785 0.0, axis 0 1 0, limit lower=-3.14 upper=3.14 effort=1.0 velocity=1.0
- added joint lm_tarsus_joint: type fixed, parent lm_tibia_link, child lm_tarsus_link, origin xyz=-0.115 0.0 0
- added joint lm_tibia_joint: type revolute, parent lm_femur_link, child lm_tibia_link, origin xyz=0.08 0.0 0.0 rpy=0 -0.785 0, axis 0 1 0, limit lower=-3.14 upper=3.14 effort=1.0 velocity=1.0
- added joint lr_coxa_joint: type revolute, parent body_link, child lr_coxa_link, origin xyz=-0.063 -0.092 0.00 rpy=0 0 -2.17, axis 0 0 1, limit lower=-3.14 upper=3.14 effort=1.0 velocity=1.0
- added joint lr_femur_joint: type revolute, parent lr_coxa_link, child lr_femur_link, origin xyz=0.022 0.00 0.00 rpy=0 -0.785 0.0, axis 0 1 0, limit lower=-3.14 upper=3.14 effort=1.0 velocity=1.0
- added joint lr_tarsus_joint: type fixed, parent lr_tibia_link, child lr_tarsus_link, origin xyz=-0.115 0.0 0
- added joint lr_tibia_joint: type revolute, parent lr_femur_link, child lr_tibia_link, origin xyz=0.08 0.0 0.0 rpy=0 -0.785 0, axis 0 1 0, limit lower=-3.14 upper=3.14 effort=1.0 velocity=1.0
- added joint rm_coxa_joint: type revolute, parent body_link, child rm_coxa_link, origin xyz=0.072 0 0.00 rpy=0 0 0, axis 0 0 1, limit lower=-3.14 upper=3.14 effort=1.0 velocity=1.0
- added joint rm_femur_joint: type revolute, parent rm_coxa_link, child rm_femur_link, origin xyz=0.022 0.00 0.00 rpy=0 -0.785 0.0, axis 0 1 0, limit lower=-3.14 upper=3.14 effort=1.0 velocity=1.0
- added joint rm_tarsus_joint: type fixed, parent rm_tibia_link, child rm_tarsus_link, origin xyz=-0.115 0.0 0
- added joint rm_tibia_joint: type revolute, parent rm_femur_link, child rm_tibia_link, origin xyz=0.08 0.0 0.0 rpy=0 -0.785 0, axis 0 1 0, limit lower=-3.14 upper=3.14 effort=1.0 velocity=1.0
- added joint rr_coxa_joint: type revolute, parent body_link, child rr_coxa_link, origin xyz=0.063 -0.092 0.00 rpy=0 0 -0.6, axis 0 0 1, limit lower=-3.14 upper=3.14 effort=1.0 velocity=1.0
- added joint rr_femur_joint: type revolute, parent rr_coxa_link, child rr_femur_link, origin xyz=0.022 0.00 0.00 rpy=0 -0.785 0.0, axis 0 1 0, limit lower=-3.14 upper=3.14 effort=1.0 velocity=1.0
- added joint rr_tarsus_joint: type fixed, parent rr_tibia_link, child rr_tarsus_link, origin xyz=-0.115 0.0 0
- added joint rr_tibia_joint: type revolute, parent rr_femur_link, child rr_tibia_link, origin xyz=0.08 0.0 0.0 rpy=0 -0.785 0, axis 0 1 0, limit lower=-3.14 upper=3.14 effort=1.0 velocity=1.0
