Commit message: Try to realise RPY, Y is work

File: goliath_description/urdf/goliath_model.xacro (robot description, xacro)
@@ -4,5 +4,6 @@
   <xacro:property name="femur_length" value="0.08" />
   <xacro:property name="tibia_length" value="0.115" />
-  <xacro:property name="leg_base_angle" value="${34.4/180*pi}" />
+  <!-- <xacro:property name="leg_base_angle" value="${34.4/180*pi}" /> -->
+  <xacro:property name="leg_base_angle" value="${45/180*pi}" />
   <xacro:property name="legs_joint_effort" value="6.0"/>
   <xacro:property name="legs_joint_velocity" value="0.524"/>
@@ -53,5 +54,5 @@
       <parent link="${side}${location}_coxa_link"/>
       <child link="${side}${location}_femur_link"/>
-      <origin xyz="${coxa_length} 0.00 0.00" rpy="0 -0.785 0.0"/>
+      <origin xyz="${coxa_length} 0.00 0.00" rpy="0 ${-pi/4} 0.0"/>
       <limit effort="${legs_joint_effort}" velocity="${legs_joint_velocity}" lower="-3.14" upper="3.14"/>
       <axis xyz="0 1 0"/>
@@ -69,5 +70,5 @@
       <parent link="${side}${location}_femur_link"/>
       <child link="${side}${location}_tibia_link"/>
-      <origin xyz="${femur_length} 0.0 0.0" rpy="0 -0.785 0"/>
+      <origin xyz="${femur_length} 0.0 0.0" rpy="0 ${-pi/4} 0"/>
       <limit effort="${legs_joint_effort}" velocity="${legs_joint_velocity}" lower="-3.14" upper="3.14"/>
       <axis xyz="0 1 0"/>
@@ -78,5 +79,5 @@
            <mesh filename="package://goliath_description/meshes/leg_end.stl" scale= "0.001 0.001 0.001" />
         </geometry>
-        <origin xyz="0.0 0.0 0.0" rpy="0 0.25 0"/>
+        <origin xyz="0.0 0.0 0.0" rpy="0 ${0.25 - pi/2} 0"/>
         <material name="rubber"/>
       </visual>
@@ -85,7 +86,8 @@
       <parent link="${side}${location}_tibia_link"/>
       <child link="${side}${location}_tarsus_link"/>
-      <origin xyz="-${tibia_length} 0.0 0"/>
+      <origin xyz="-${tibia_length} 0.0 0" rpy="0 ${pi/2} 0"/>
     </joint>
   </xacro:macro>
+s
   <xacro:leg side="l" location="f" x="-0.063" y="0.092"  angle="${pi - leg_base_angle}" />
   <xacro:leg side="l" location="m" x="-0.072" y="0"      angle="${pi}" />

Commit message: Refactoring of teleop_key.cpp

File: goliath_description/urdf/goliath_model.xacro (robot description, xacro)
@@ -4,6 +4,5 @@
   <xacro:property name="femur_length" value="0.08" />
   <xacro:property name="tibia_length" value="0.115" />
-  <!-- <xacro:property name="leg_base_angle" value="${34.4/180*pi}" /> -->
-  <xacro:property name="leg_base_angle" value="${45/180*pi}" />
+  <xacro:property name="leg_base_angle" value="${34.4/180*pi}" />
   <xacro:property name="legs_joint_effort" value="6.0"/>
   <xacro:property name="legs_joint_velocity" value="0.524"/>
@@ -39,5 +38,5 @@
       <child link="${side}${location}_coxa_link"/>
       <origin xyz="${x} ${y} 0.00" rpy="0 0 ${angle}"/>
-      <limit effort="${legs_joint_effort}" velocity="${legs_joint_velocity}" lower="-3.14" upper="3.14"/>
+      <limit effort="${legs_joint_effort}" velocity="${legs_joint_velocity}" lower="-0.93" upper="0.93"/>
       <axis xyz="0 0 1"/>
     </joint>
@@ -55,5 +54,5 @@
       <child link="${side}${location}_femur_link"/>
       <origin xyz="${coxa_length} 0.00 0.00" rpy="0 ${-pi/4} 0.0"/>
-      <limit effort="${legs_joint_effort}" velocity="${legs_joint_velocity}" lower="-3.14" upper="3.14"/>
+      <limit effort="${legs_joint_effort}" velocity="${legs_joint_velocity}" lower="-0.88" upper="2.27"/>
       <axis xyz="0 1 0"/>
     </joint>
@@ -71,5 +70,5 @@
       <child link="${side}${location}_tibia_link"/>
       <origin xyz="${femur_length} 0.0 0.0" rpy="0 ${-pi/4} 0"/>
-      <limit effort="${legs_joint_effort}" velocity="${legs_joint_velocity}" lower="-3.14" upper="3.14"/>
+      <limit effort="${legs_joint_effort}" velocity="${legs_joint_velocity}" lower="-2.6" upper="0.44"/>
       <axis xyz="0 1 0"/>
     </joint>

Commit message: Change X and Y axis

File: goliath_description/urdf/goliath_model.xacro (robot description, xacro)
@@ -4,5 +4,5 @@
   <xacro:property name="femur_length" value="0.08" />
   <xacro:property name="tibia_length" value="0.115" />
-  <xacro:property name="leg_base_angle" value="${34.4/180*pi}" />
+  <xacro:property name="leg_base_angle" value="${55.6/180*pi}" />
   <xacro:property name="legs_joint_effort" value="6.0"/>
   <xacro:property name="legs_joint_velocity" value="0.524"/>
@@ -19,5 +19,5 @@
         <mesh filename="package://goliath_description/meshes/body.stl" scale= "0.001 0.001 0.001" />
       </geometry>
-      <origin xyz="0.0 0.0 0.0448" rpy="0 0 0"/>
+      <origin xyz="0.0 0.0 0.0448" rpy="0 0 ${-pi/2}"/>
       <material name="alumunium"/>
     </visual>
@@ -88,10 +88,9 @@
     </joint>
   </xacro:macro>
-s
-  <xacro:leg side="l" location="f" x="-0.063" y="0.092"  angle="${pi - leg_base_angle}" />
-  <xacro:leg side="l" location="m" x="-0.072" y="0"      angle="${pi}" />
-  <xacro:leg side="l" location="r" x="-0.063" y="-0.092" angle="${-(pi - leg_base_angle)}" />
-  <xacro:leg side="r" location="f" x="0.063"  y="0.092"  angle="${leg_base_angle}" />
-  <xacro:leg side="r" location="m" x="0.072"  y="0"      angle="${0}" />
-  <xacro:leg side="r" location="r" x="0.063"  y="-0.092" angle="-${leg_base_angle}" />
+  <xacro:leg side="l" location="f" x="0.092"  y="0.063"   angle="${leg_base_angle}" />
+  <xacro:leg side="l" location="m" x="0"      y="0.072"   angle="${pi/2}" />
+  <xacro:leg side="l" location="r" x="-0.092" y="0.063"   angle="${pi - leg_base_angle}" />
+  <xacro:leg side="r" location="f" x="0.092"  y="-0.063"  angle="${-leg_base_angle}" />
+  <xacro:leg side="r" location="m" x="0"      y="-0.072"  angle="${-pi/2}" />
+  <xacro:leg side="r" location="r" x="-0.092" y="-0.063"  angle="${-pi + leg_base_angle}" />
 </robot>
